Commit message: Add files via upload

File: quadruped/resources/custom_robot.urdf (robot description, URDF)
Before this commit: robot quadruped, 19 links, 18 joints
Joints:
- joint head-flange1: limit lower=-0.5 upper=0.5 effort=10 velocity=10 -> lower=-0.2 upper=0.5 effort=10 velocity=10
- joint head-flange2: limit lower=-0.5 upper=0.5 effort=10 velocity=10 -> lower=-0.2 upper=0.5 effort=10 velocity=10
- joint tail-flange3: limit lower=-0.5 upper=0.5 effort=10 velocity=10 -> lower=-0.2 upper=0.5 effort=10 velocity=10
- joint tail-flange4: limit lower=-0.5 upper=0.5 effort=10 velocity=10 -> lower=-0.2 upper=0.5 effort=10 velocity=10
